File: board/hitem.sch (KiCad schematic (older format))
At the start: 59 parts, among them J1 CONN_02X04

Commit message: Change the design to be based on RedBearLab WiFi Micro
Parts:
- removed C?: 0.1u, symbol C
- removed J?: CONN_01X05, symbol CONN_01X05
- removed J?: CONN_02X03, symbol CONN_02X03
- removed L?: 4.7uH, symbol INDUCTOR
- removed R?: 100K, symbol R
- removed U?: TPS61222DCKR, symbol TPS61220
- removed U?: PIC16LF1713-I/SO, symbol PIC16Lx1713_6_8_SOIC
- added J5, J6: Female, 0.1\", 1x10, symbol CONN_01X10
- added L1: B82462G4472M, avishay:B82462G4472M, symbol B82462G4472M
- added R14: 1.6M, avishay:R0603, symbol R
- added R15, R17: 180K, avishay:R0603, symbol R
- added U1: TPS61070, avishay:TPS61070DDCR, symbol TPS6107x
- C1, C2, C3, C4, C5, C6, C7, C8, C9: renamed from C?; footprint (none) -> Avishay:R0603
- D1, D6, D7: renamed from D?; footprint (none) -> avishay:SOD-523F
- D2, D3, D4, D5: renamed from D?; footprint (none) -> Avishay:LED_RGB_TH_5MM
- J1: value CONN_02X04 -> Male, 0.1\", 2x4
- J2: renamed from J?; value CONN_01X02 -> Male, 0.1\", 1x2
- J3: renamed from P?; value CONN_02X05 -> Female, 0.1\", 2x5
- J4: renamed from J?; value CONN_02X02 -> Male, 0.1\", 2x2
- Q1, Q2, Q3, Q4, Q5: renamed from Q?; footprint (none) -> avishay:BSS214NH6327
- Q6: renamed from Q?; footprint (none) -> avishay:R0603
- R1, R10, R11, R12, R13, R16, R2, R20, R22, R23, R24, R26, R28, R3, R4, R8, R9: renamed from R?; footprint (none) -> avishay:R0603
- R18, R19: renamed from R?; value 100K -> 180K; footprint (none) -> avishay:R0603
- R21, R25, R27, R5, R6, R7: renamed from R?; value 2M -> 1.6M; footprint (none) -> avishay:R0603
- U2: renamed from U?; footprint (none) -> avishay:LIS2HH12
Connections:
- net labels removed: ICSPCLK, ICSPDAT, MCLR
- wire segments 205 -> 180
Other:
- note added: "IO23_D8\nIO29_D9\nNRST\nIO11_D14\nIO10_D15\nIO3_A3\nIO4_A2\nIO5_A1\n3V3\nGND"
- note added: "IO8_D7\nIO24_D6\nIO9_D5\nIO17_D4\nIO16_D22\nIO15_D23\nIO14_D24\nIO7_D3\nIO6_D2\nIO1_D1\nIO2_D0"
- note added: "RedBearLab WiFi Micro"
- note removed: "Programming\nConnector"
- moved on the sheet: C3, D6, D7, J4, R16, R18, R19, R22, R23

Commit message: Final version of schematic & PCB
Parts:
- C1, C2, C3, C4, C5, C6, C7, C8, C9: footprint Avishay:R0603 -> avishay:R0603
- D2, D3, D4, D5: footprint Avishay:LED_RGB_TH_5MM -> avishay:LED_RGB_TH_5MM
- J1: footprint (none) -> Pin_Headers:Pin_Header_Straight_2x04
- J2: footprint (none) -> Pin_Headers:Pin_Header_Straight_2x01
- J3: footprint (none) -> Pin_Headers:Pin_Header_Straight_2x05
- J4: footprint (none) -> Pin_Headers:Pin_Header_Straight_2x02
- J5, J6: footprint (none) -> Pin_Headers:Pin_Header_Straight_1x10
- Q6: footprint avishay:R0603 -> avishay:BSS214NH6327
Connections:
- wire segments 180 -> 182
Other:
- moved on the sheet: C8, C9, R28
Changed lines of the file:
@@
 LIBS:valves
 LIBS:avishay
+LIBS:hitem
 LIBS:hitem-cache
 EELAYER 25 0
@@
 F 0 "J1" H 2150 1000 50  0000 C CNN
 F 1 "Male, 0.1\", 2x4" H 2100 900 50  0000 C CNN
-F 2 "" H 2150 100 50  0001 C CNN
+F 2 "Pin_Headers:Pin_Header_Straight_2x04" H 2150 100 50  0001 C CNN
 F 3 "" H 2150 100 50  0000 C CNN
 	1    2150 1300
@@
 F 0 "D3" H 3175 4000 50  0000 C CNN
 F 1 "LED_RABG" H 3125 3300 50  0000 C CNN
-F 2 "Avishay:LED_RGB_TH_5MM" H 3050 3600 50  0001 C CNN
+F 2 "avishay:LED_RGB_TH_5MM" H 3050 3600 50  0001 C CNN
 F 3 "" H 3050 3600 50  0000 C CNN
 	1    3100 3650
@@
 F 0 "D2" H 3175 3150 50  0000 C CNN
 F 1 "LED_RABG" H 3125 2450 50  0000 C CNN
-F 2 "Avishay:LED_RGB_TH_5MM" H 3050 2750 50  0001 C CNN
+F 2 "avishay:LED_RGB_TH_5MM" H 3050 2750 50  0001 C CNN
 F 3 "" H 3050 2750 50  0000 C CNN
 	1    3100 2800
@@
 F 0 "D4" H 3175 4850 50  0000 C CNN
 F 1 "LED_RABG" H 3125 4150 50  0000 C CNN
-F 2 "Avishay:LED_RGB_TH_5MM" H 3050 4450 50  0001 C CNN
+F 2 "avishay:LED_RGB_TH_5MM" H 3050 4450 50  0001 C CNN
 F 3 "" H 3050 4450 50  0000 C CNN
 	1    3100 4500
@@
 F 0 "D5" H 3175 5700 50  0000 C CNN
 F 1 "LED_RABG" H 3125 5000 50  0000 C CNN
-F 2 "Avishay:LED_RGB_TH_5MM" H 3050 5300 50  0001 C CNN
+F 2 "avishay:LED_RGB_TH_5MM" H 3050 5300 50  0001 C CNN
 F 3 "" H 3050 5300 50  0000 C CNN
 	1    3100 5350
@@
 F 0 "J2" H 750 6950 50  0000 C CNN
 F 1 "Male, 0.1\", 1x2" V 850 6800 50  0001 C CNN
-F 2 "" H 750 6800 50  0001 C CNN
+F 2 "Pin_Headers:Pin_Header_Straight_2x01" H 750 6800 50  0001 C CNN
 F 3 "" H 750 6800 50  0000 C CNN
 	1    750  6800
@@
 F 0 "Q6" H 7950 2150 50  0000 R CNN
 F 1 "BSS214N" H 8200 2050 50  0000 R CNN
-F 2 "avishay:R0603" H 7850 2200 50  0001 C CNN
+F 2 "avishay:BSS214NH6327" H 7850 2200 50  0001 C CNN
 F 3 "" H 7650 2100 50  0000 C CNN
 F 4 "726-BSS214NH6327XT" H 7650 2100 60  0001 C CNN "mouser"
@@
 F 0 "J3" V 5100 1650 50  0000 C CNN
 F 1 "Female, 0.1\", 2x5" V 5200 1950 50  0000 C CNN
-F 2 "" H 5150 100 50  0001 C CNN
+F 2 "Pin_Headers:Pin_Header_Straight_2x05" H 5150 100 50  0001 C CNN
 F 3 "" H 5150 100 50  0000 C CNN
 	1    5150 1300
@@
 F 0 "C1" H 1700 7050 50  0000 L CNN
 F 1 "10uF" H 1700 6950 50  0000 L CNN
-F 2 "Avishay:R0603" H 1550 7000 50  0001 C CNN
+F 2 "avishay:R0603" H 1550 7000 50  0001 C CNN
 F 3 "" H 1550 7000 50  0000 C CNN
 	1    1550 7000
@@
 F 0 "C3" H 3350 6700 50  0000 L CNN
 F 1 "10uF" H 3300 6600 50  0000 L CNN
-F 2 "Avishay:R0603" H 3550 6800 50  0001 C CNN
+F 2 "avishay:R0603" H 3550 6800 50  0001 C CNN
 F 3 "" H 3550 6800 50  0000 C CNN
 	1    3550 6800
@@
 	1    8950 2500
 	1    0    0    -1
-$EndComp
-$Comp
-L +BATT #PWR013
-U 1 1 56BD4161
-P 8600 1700
-F 0 "#PWR013" H 8600 1550 50  0001 C CNN
-F 1 "+BATT" H 8600 1840 50  0000 C CNN
-F 2 "" H 8600 1700 50  0000 C CNN
-F 3 "" H 8600 1700 50  0000 C CNN
-	1    8600 1700
-	0    -1   -1   0
 $EndComp
 $Comp
@@
 L R R28
 U 1 1 56BD4A1B
-P 8800 1700
-F 0 "R28" V 8600 1700 50  0000 C CNN
-F 1 "0" V 8700 1700 50  0000 C CNN
-F 2 "avishay:R0603" V 8730 1700 50  0001 C CNN
-F 3 "" H 8800 1700 50  0000 C CNN
-	1    8800 1700
+P 9800 750
+F 0 "R28" V 9600 750 50  0000 C CNN
+F 1 "0" V 9700 750 50  0000 C CNN
+F 2 "avishay:R0603" V 9730 750 50  0001 C CNN
+F 3 "" H 9800 750 50  0000 C CNN
+	1    9800 750
 	0    1    1    0
 $EndComp
@@
 L C C8
 U 1 1 56BDDE4F
-P 9550 900
-F 0 "C8" H 9300 950 50  0000 L CNN
-F 1 "0.1u" H 9250 850 50  0000 L CNN
-F 2 "Avishay:R0603" H 9588 750 50  0001 C CNN
-F 3 "" H 9550 900 50  0000 C CNN
-	1    9550 900
-	1    0    0    -1
+P 9450 900
+F 0 "C8" H 9200 950 50  0000 L CNN
+F 1 "0.1u" H 9150 850 50  0000 L CNN
+F 2 "avishay:R0603" H 9488 750 50  0001 C CNN
+F 3 "" H 9450 900 50  0000 C CNN
+	1    9450 900
+	-1   0    0    -1
 $EndComp
 $Comp
 L C C9
 U 1 1 56BDDF6C
-P 9950 900
-F 0 "C9" H 10100 950 50  0000 L CNN
-F 1 "0.1u" H 10100 850 50  0000 L CNN
-F 2 "Avishay:R0603" H 9988 750 50  0001 C CNN
-F 3 "" H 9950 900 50  0000 C CNN
-	1    9950 900
-	1    0    0    -1
+P 9050 900
+F 0 "C9" H 9200 950 50  0000 L CNN
+F 1 "0.1u" H 9200 850 50  0000 L CNN
+F 2 "avishay:R0603" H 9088 750 50  0001 C CNN
+F 3 "" H 9050 900 50  0000 C CNN
+	1    9050 900
+	-1   0    0    -1
 $EndComp
 $Comp
 L +BATT #PWR014
 U 1 1 56BDE9B6
-P 9350 700
-F 0 "#PWR014" H 9350 550 50  0001 C CNN
-F 1 "+BATT" H 9350 840 50  0000 C CNN
-F 2 "" H 9350 700 50  0000 C CNN
-F 3 "" H 9350 700 50  0000 C CNN
-	1    9350 700
-	1    0    0    -1
+P 10150 750
+F 0 "#PWR014" H 10150 600 50  0001 C CNN
+F 1 "+BATT" H 10150 890 50  0000 C CNN
+F 2 "" H 10150 750 50  0000 C CNN
+F 3 "" H 10150 750 50  0000 C CNN
+	1    10150 750
+	-1   0    0    -1
 $EndComp
 $Comp
 L GND #PWR015
 U 1 1 56BDEC0D
-P 9550 1150
-F 0 "#PWR015" H 9550 900 50  0001 C CNN
-F 1 "GND" H 9550 1000 50  0000 C CNN
-F 2 "" H 9550 1150 50  0000 C CNN
-F 3 "" H 9550 1150 50  0000 C CNN
-	1    9550 1150
-	1    0    0    -1
+P 9450 1150
+F 0 "#PWR015" H 9450 900 50  0001 C CNN
+F 1 "GND" H 9450 1000 50  0000 C CNN
+F 2 "" H 9450 1150 50  0000 C CNN
+F 3 "" H 9450 1150 50  0000 C CNN
+	1    9450 1150
+	-1   0    0    -1
 $EndComp
 $Comp
@@
 F 0 "C4" H 3850 3200 50  0000 L CNN
 F 1 "1uF" H 3850 3100 50  0000 L CNN
-F 2 "Avishay:R0603" H 3788 2850 50  0001 C CNN
+F 2 "avishay:R0603" H 3788 2850 50  0001 C CNN
 F 3 "" H 3750 3000 50  0000 C CNN
 	1    3750 3000
@@
 F 0 "C2" V 2100 850 50  0000 L CNN
 F 1 "1uF" V 2000 850 50  0000 L CNN
-F 2 "Avishay:R0603" H 2188 550 50  0001 C CNN
+F 2 "avishay:R0603" H 2188 550 50  0001 C CNN
 F 3 "" H 2150 700 50  0000 C CNN
 	1    2150 700
@@
 F 0 "C5" H 3850 4050 50  0000 L CNN
 F 1 "1uF" H 3850 3950 50  0000 L CNN
-F 2 "Avishay:R0603" H 3788 3700 50  0001 C CNN
+F 2 "avishay:R0603" H 3788 3700 50  0001 C CNN
 F 3 "" H 3750 3850 50  0000 C CNN
 	1    3750 3850
@@
 F 0 "C6" H 3850 4900 50  0000 L CNN
 F 1 "1uF" H 3850 4800 50  0000 L CNN
-F 2 "Avishay:R0603" H 3788 4550 50  0001 C CNN
+F 2 "avishay:R0603" H 3788 4550 50  0001 C CNN
 F 3 "" H 3750 4700 50  0000 C CNN
 	1    3750 4700
@@
 F 0 "C7" H 3850 5700 50  0000 L CNN
 F 1 "1uF" H 3850 5600 50  0000 L CNN
-F 2 "Avishay:R0603" H 3788 5350 50  0001 C CNN
+F 2 "avishay:R0603" H 3788 5350 50  0001 C CNN
 F 3 "" H 3750 5500 50  0000 C CNN
 	1    3750 5500
@@
 F 0 "J4" H 6250 6900 50  0000 C CNN
 F 1 "Male, 0.1\", 2x2" H 6300 6800 50  0001 C CNN
-F 2 "" H 6250 5850 50  0001 C CNN
+F 2 "Pin_Headers:Pin_Header_Straight_2x02" H 6250 5850 50  0001 C CNN
 F 3 "" H 6250 5850 50  0000 C CNN
 	1    6250 7050
@@
 F 0 "J5" H 6800 5050 50  0000 C CNN
 F 1 "Female, 0.1\", 1x10" V 6900 4500 50  0001 C CNN
-F 2 "" H 6800 4500 50  0001 C CNN
+F 2 "Pin_Headers:Pin_Header_Straight_1x10" H 6800 4500 50  0001 C CNN
 F 3 "" H 6800 4500 50  0000 C CNN
 	1    6800 4500
@@
 F 0 "J6" H 8450 5050 50  0000 C CNN
 F 1 "Female, 0.1\", 1x10" V 8550 4500 50  0001 C CNN
-F 2 "" H 8450 4500 50  0001 C CNN
+F 2 "Pin_Headers:Pin_Header_Straight_1x10" H 8450 4500 50  0001 C CNN
 F 3 "" H 8450 4500 50  0000 C CNN
 	1    8450 4500
@@
 	2350 4650 2500 4650
 Wire Wire Line
-	2350 3650 2600 3650
+	2350 3650 2800 3650
 Wire Wire Line
 	2350 2600 2800 2600
@@
 Wire Wire Line
 	9100 1800 9100 1700
-Wire Wire Line
-	8950 1700 9150 1700
 Connection ~ 9100 1700
 Wire Wire Line
@@
 	1400 6350 1400 6750
 Wire Wire Line
-	8650 1700 8600 1700
+	10400 1000 10350 1000
 Wire Wire Line
 	10350 1700 11000 1700
@@
 	10350 2300 11000 2300
 Wire Wire Line
-	9350 750  9950 750
-Wire Wire Line
-	9350 750  9350 700
-Connection ~ 9550 750
-Wire Wire Line
-	9550 1050 9550 1150
-Wire Wire Line
-	9550 1100 9950 1100
-Wire Wire Line
-	9950 1100 9950 1050
-Connection ~ 9550 1100
+	9650 750  9050 750
+Connection ~ 9450 750
+Wire Wire Line
+	9450 1050 9450 1150
+Wire Wire Line
+	9450 1100 9050 1100
+Wire Wire Line
+	9050 1050 9050 1700
+Connection ~ 9450 1100
 Wire Wire Line
 	1200 1150 1200 1300
@@
 7C 87 17 6E 00 50 C3 D4 30 09 60 2A 65 E7 BC 16 A7 CA C5 E9 9F 9C BD F7 96 D2 06 ED D9 9B 9A 75
 A6 7B D5 D8 F8 1A 00 F8 12 4C F5 FC 66 94 CD EA AF 90 8A 5A B6 E6 89 5F 09 94 2F 21 5C FC 3F 42
-69 C5 EF EA F3 3C 51 00 00 00 00 49 45 4E 44 AE 42 60 82 F3
+69 C5 EF EA F3 3C 51 00 00 00 00 49 45 4E 44 AE 42 60 82 33
 EndData
 $EndBitmap
@@
 Wire Wire Line
 	1450 6500 1400 6500
+$Comp
+L LOGO #G?
+U 1 1 56CDE3B9
+P 9500 5900
+F 0 "#G?" H 9500 5584 60  0001 C CNN
+F 1 "LOGO" H 9500 6216 60  0001 C CNN
+F 2 "" H 9500 5900 60  0000 C CNN
+F 3 "" H 9500 5900 60  0000 C CNN
+	1    9500 5900
+	1    0    0    -1
+$EndComp
+Wire Wire Line
+	8650 4850 9200 4850
+Wire Wire Line
+	8650 4950 9200 4950
+Text Label 8700 4850 0    60   ~ 0
+ACCEL_INT1
+Text Label 8700 4950 0    60   ~ 0
+ACCEL_INT2
+Wire Wire Line
+	9050 1700 9150 1700
+Connection ~ 9050 1100
+Wire Wire Line
+	10150 750  9950 750
 $EndSCHEMATC

Commit message: Schematic for rev B
Parts:
- removed C1, C3: 10uF, avishay:R0603, symbol CP1
- removed C2: 1uF, avishay:R0603, symbol C
- removed C9: 0.1u, avishay:R0603, symbol C
- removed D2, D3, D4, D5: LED_RABG, avishay:LED_RGB_TH_5MM, symbol LED_RABG
- removed D6, D7: CDBU0130L, avishay:SOD-523F, symbol D_Schottky_Small
- removed J1: Male, 0.1\", 2x4, Pin_Headers:Pin_Header_Straight_2x04, symbol CONN_02X04
- removed J2: Male, 0.1\", 1x2, Pin_Headers:Pin_Header_Straight_2x01, symbol CONN_01X02
- removed J3: Female, 0.1\", 2x5, Pin_Headers:Pin_Header_Straight_2x05, symbol CONN_02X05
- removed J4: Male, 0.1\", 2x2, Pin_Headers:Pin_Header_Straight_2x02, symbol CONN_02X02
- removed L1: B82462G4472M, avishay:B82462G4472M, symbol B82462G4472M
- removed Q3, Q5, Q6: BSS214N, avishay:BSS214NH6327, symbol Q_NMOS_GSD
- removed R11, R12, R13: 50, avishay:R0603, symbol R
- removed R15: 180K, avishay:R0603, symbol R
- removed R16: 0, avishay:R0603, symbol R
- removed R2, R24, R26: 1K, avishay:R0603, symbol R
- removed R22, R23: 100K, avishay:R0603, symbol R
- removed R25, R27: 1.6M, avishay:R0603, symbol R
- removed U1: TPS61070, avishay:TPS61070DDCR, symbol TPS6107x
- removed U2: LIS2HH12TR, avishay:LIS2HH12, symbol LIS2HH12TR
- added C1, C3, C8: 1uF, avishay:R0603, symbol C
- added J3: Header, .100\", symbol CONN_02X02
- added J4: CONN_01X03, symbol CONN_01X03
- added J5: Header, .100\", symbol CONN_02X06
- added J6, J7: CONN_01X01, symbol CONN_01X01
- added U1: LIS3DH, symbol LIS3DH
- added U2: XC6120, symbol XC6120
- added U3, U4, U7, U8: WS2812B, symbol WS2812B
- added U5: SPARKFUN_LIS3DH, symbol SPARKFUN_LIS3DH
- added U6: MIC5255, symbol MIC5255
- C7: value 1uF -> 0.01uF; footprint avishay:R0603 -> (none)
- R1: value 0 -> 1K
- R10: value 50 -> 180K
- R14: value 1.6M -> 1K
- R3: value 1K -> 1.6M
- R4: value 1K -> 47K
- R5, R6, R7: value 1.6M -> 0
- R8, R9: value 50 -> 0
- renumbered C8 to C2, J5 to J1, J6 to J2, Q4 to Q3, R17 to R11, R18 to R12, R19 to R13, R20 to R15, R21 to R16, R28 to R2
Connections:
- net labels added: +3.3V, ACCEL_INT, AUX1, AUX2, AUX3, LED, RX1, TX1
- net labels removed: +5V, ACCEL_INT1, ACCEL_INT2, LD2, LD3, LED1, LED2, LED3, NRF_CE, NRF_CS, NRF_INT, PIEZO1, PIEZO2, VBAT
- wire segments 182 -> 170
Other:
- note added: "AUX\nConnector"
- note added: "BATT+"
- note added: "BATT-"
- note added: "CC-BY-SA"
- note added: "Ext.\nLEDs"
- note added: "IO23_D8\nIO29_D9\nNRST\nIO11_D14\nIO10_D15\nIO3_A3\nIO4_A2\nIO5_A1\n3V3\nGND\nVIN"
- note added: "OPTION A: On-Board Accelerometer"
- note added: "OPTION B: Sparkfun Module SEN-13963"
- note added: "Power"
- note added: "Protection\nBypass"
- note added: "R4..R8 - Bypass for individual LEDs"
- note removed: "Auxiliary Load Switches"
- note removed: "IO23_D8\nIO29_D9\nNRST\nIO11_D14\nIO10_D15\nIO3_A3\nIO4_A2\nIO5_A1\n3V3\nGND"
- note removed: "NRF Board Connector"
- note removed: "Piezo Interface"
- note removed: "Power Supply"
- moved on the sheet: C2, D1, J1, J2, Q3, R11, R12, R13, R15, R16, R2

Commit message: Finish schematic & board layout (without routing)
Parts:
- added C9: 1uF, avishay:R0603, symbol C
- C7: footprint (none) -> avishay:R0603
- J3: footprint (none) -> Pin_Headers:Pin_Header_Straight_2x02
- J4: footprint (none) -> avishay:SMT_HOOKUP_3
- J5: footprint (none) -> Pin_Headers:Pin_Header_Straight_2x06
- J6, J7: footprint (none) -> hitem:BATTERY_CONTACT
- Q1, Q2, Q3: footprint avishay:BSS214NH6327 -> avishay:SOT-23
- U1: footprint (none) -> hitem:LIS3DH
- U2: footprint (none) -> hitem:XC6221
- U3, U4, U7, U8: footprint (none) -> hitem:WS2812
- U5: footprint (none) -> avishay:SEN-13963
- U6: footprint (none) -> hitem:MIC5255
Connections:
- wire segments 170 -> 165
Other:
- moved on the sheet: C4, C5, C6, C8
